File: routed/keyboard-left.kicad_pcb (KiCad board)
At the start: 2 copper layers, 144.2 x 128.6 mm, 62 parts, among them P1 C1, P10 R2, P11 R3, P12 R4, P13 R5, P14 R6, P15 R7, P16 R8, P17 D1, P2 C2, P3 C3, P4 C4, P5 C5, P6 C6, P7 C7, P8 C8, P9 R1

Commit message: feat(route): fresh freerouting baseline for the bottom-side layout
Supersedes the bay-era baseline: 1231 segments, 167 vias, 8
unconnected items (~95%) on the compact placement. Same finishing
list as before: USB D+/- pair by hand, power tree at 0.4mm, tie off
the GND stubs and leftover switch nets, DRC clean before gerbers.
Parts:
- moved P2 85.1 mm to (158.6, 104.5), turned to 90 degrees
- moved P1 84.3 mm to (158.6, 101.0), turned to 90 degrees
- moved P3 82.4 mm to (168.4, 100.5)
- moved P4 78.7 mm to (171.5, 104.8), turned to 0 degrees
- moved P13 75.0 mm to (163.9, 96.3)
- moved P17 74.9 mm to (167.5, 96.3), turned to 0 degrees
- moved 19.056 74.7 mm to (163.5, 100.0)
- moved 19.057 74.7 mm to (171.5, 100.0)
- moved P5 69.7 mm to (171.5, 96.3), turned to 0 degrees
- moved P7 64.3 mm to (188.0, 45.1)
- moved 19.052 51.3 mm to (181.5, 47.0)
- moved P14 50.5 mm to (170.8, 88.0), turned to 90 degrees
- moved 19.053 49.4 mm to (163.5, 85.0)
- moved P8 49.3 mm to (169.8, 83.1)
- moved P16 49.0 mm to (159.5, 96.3)
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Routing:
- net sw_matrix_outer_bottom: track 10.3 -> 139.1 mm, vias 1 -> 3
- net sw_matrix_outer_home: track 138.3 -> 10.6 mm, vias 2 -> 1
- net sw_matrix_pinky_bottom: track 10.6 -> 118.2 mm, vias 1 -> 3
- net sw_matrix_inner_bottom: track 123.0 -> 54.6 mm, vias 4 -> 3
- net sw_matrix_outer_num: track 90.6 -> 149.3 mm, vias 1 -> 2
- net USB_DM: track 76.0 -> 17.5 mm, vias 4 -> 2
- net sw_thumbs_space_cluster: track 132.4 -> 74.6 mm, vias 4 -> 1
- net VBAT: track 128.7 -> 71.8 mm, vias 8 -> 4
- net ENC_SW: track 90.1 -> 35.4 mm, vias 1 -> 0
- net sw_thumbs_layer_cluster: track 112.7 -> 59.8 mm, vias 2 -> 1
- net sw_matrix_pinky_num: track 82.2 -> 134.3 mm, vias 2 -> 4
- net sw_matrix_outer_top: track 120.3 -> 172.0 mm
- net sw_matrix_middle_num: track 33.1 -> 82.1 mm
- net sw_matrix_ring_num: track 54.0 -> 102.7 mm, vias 3 -> 4
- net sw_matrix_pinky_top: track 98.0 -> 144.5 mm, vias 4 -> 2
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Other:
- board size 144.2 x 128.6 mm -> 144.2 x 122.6 mm

Commit message: feat(route): autoroute baseline for the flattened outline
Replaces the stale pre-flatten baseline. Hand-finish list unchanged:
USB D+/- pair, power tree at 0.4mm, GND stubs + leftover switch nets,
DRC clean before gerbers.
Parts:
- moved P11 56.4 mm to (182.4, 92.5)
- moved P12 56.4 mm to (182.4, 95.5)
- moved 19.054 55.7 mm to (188.0, 95.0), turned to 90 degrees
- moved 19.055 43.9 mm to (180.5, 98.5)
- moved 19.052 39.8 mm to (176.5, 86.5)
- moved DISP1 38.2 mm to (181.6, 87.7)
- moved P7 32.3 mm to (177.2, 75.5), turned to 0 degrees
- moved P9 17.4 mm to (170.4, 77.0)
- moved P10 16.9 mm to (170.4, 80.0)
- moved P15 12.0 mm to (175.4, 73.3)
- moved P17 9.53 mm to (170.0, 105.5)
- moved 19.051 9.01 mm to (173.3, 62.1), turned to -8 degrees
- moved P6 6.61 mm to (165.9, 72.0)
- moved P14 0.40 mm to (170.4, 88.0)
Routing:
- net sw_matrix_outer_home: track 10.6 -> 136.0 mm, vias 1 -> 4
- net GND: track 845.7 -> 783.2 mm
- net sw_matrix_pinky_home: track 164.1 -> 114.0 mm
- net sw_matrix_inner_top: track 83.6 -> 34.6 mm, vias 4 -> 3
- net USB_DM: track 17.5 -> 64.5 mm, vias 2 -> 4
- net SPI_SCK: track 22.3 -> 59.8 mm, vias 1 -> 2
- net SPI_MOSI: track 17.8 -> 55.0 mm, vias 1 -> 2
- net sw_matrix_middle_home: track 104.2 -> 67.5 mm, vias 3 -> 4
- net sw_matrix_outer_top: track 172.0 -> 137.8 mm, vias 3 -> 2
- net USB_DP: track 38.3 -> 72.1 mm
- net sw_matrix_ring_top: track 124.8 -> 92.3 mm
- net NV_CS: track 29.1 -> 60.3 mm, vias 1 -> 2
- net sw_matrix_ring_home: track 126.6 -> 96.3 mm, vias 7 -> 5
- net sw_matrix_index_top: track 90.1 -> 60.5 mm
- net sw_matrix_middle_top: track 97.1 -> 71.7 mm, vias 3 -> 2
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Other:
- board size 144.2 x 122.6 mm -> 144.2 x 110.9 mm
